File: ESP32S3_Carrier.kicad_pcb (KiCad board)
At the start: 2 copper layers, 116 x 170 mm, 67 parts, among them J1 CC1101 433MHz SMA, J2 NRF24L01+PA+LNA #1, J3 NRF24L01+PA+LNA #2, J4 PN532 V3 (I2C), J5 OLED 1.3in SH1106 I2C, J6 Catalex microSD, J7 RDM6300 125kHz, J8 125kHz coil, J9 Si5351 clock gen (3x SMA), Q1 PN2222A, Q2 PN2222A, Q3 AO3401A, SW1 UP, SW2 DOWN, SW3 LEFT, SW4 RIGHT, SW5 OK, SW6 BACK, SW7 MODULE PWR, U1 ESP32-S3-DevKitC-1 N16R8, U2 AMS1117-3.3, U3 VS1838B

Commit message: IR LED resistors 33R -> 47R, README notes
- 47R per IR LED (~67 mA, ~0.21 W) so a stuck-high IO2 stays inside the 1206 rating
- README: drive IO2 only with the 38 kHz carrier; how to handle starved_thermal after a re-route

Co-Authored-By: Claude Opus 5.5 <noreply@anthropic.com>
Claude-Session: https://claude.ai/code/session_01M7B8FMVeVb1bqPRBZwSV29
Parts:
- R17, R18, R5: value 33 -> 47

Commit message: Si5351: match the real 7-pin module (30.7x21.6 mm)
- 1x7 socket: 0, 1, 2, SCL, SDA, GND, VIN (VIN square pad), header 2.2 mm from the edge, centred
- Only SCL/SDA/GND/VIN connected; VIN on +3V3_MOD (module level shifter pulls I2C to VIN)
- CC1101 2x4 orientation confirmed by the owner
- Re-routed: ERC 0/0, DRC 0 (schematic parity), 277 stitching vias

Co-Authored-By: Claude Opus 5.5 <noreply@anthropic.com>
Claude-Session: https://claude.ai/code/session_01M7B8FMVeVb1bqPRBZwSV29
Parts:
- moved C17 18.1 mm to (129.4, 180.8)
- moved J9 5.24 mm to (144.6, 187.6)
Connections:
- J9 pad 1: +3V3_MOD -> unconnected-(J9-CLK0-Pad1)
- J9 pad 2: GND -> unconnected-(J9-CLK1-Pad2)
- J9 pad 3: /I2C_SCL -> unconnected-(J9-CLK2-Pad3)
- J9 pad 4: /I2C_SDA -> /I2C_SCL
Routing:
- net GND: track 651.4 -> 624.5 mm, vias 245 -> 279
- net /NRF1_IRQ: track 162.2 -> 139.3 mm, vias 1 -> 0
- net /IR_TX: track 130.8 -> 118.0 mm
- net /CC_GDO0: track 123.9 -> 133.2 mm
- net /CC_GDO2: track 90.6 -> 98.3 mm, vias 0 -> 1
- net +3V3_MOD: track 365.2 -> 358.3 mm, vias 3 -> 4
- net /BTN_RIGHT: track 41.0 -> 45.9 mm
- net /SPI_MISO: track 235.3 -> 239.4 mm, vias 3 -> 1
- net /BTN_LEFT: track 64.5 -> 68.4 mm
- net /SPI_MOSI: track 226.2 -> 230.1 mm, vias 4 -> 2
- net +5V_MOD: track 322.6 -> 318.8 mm
- net /I2C_SCL: track 204.0 -> 200.8 mm, vias 1 -> 3
- net /SPI_SCK: track 221.9 -> 225.1 mm, vias 2 -> 5
- net /BTN_DOWN: track 39.1 -> 41.8 mm
- net /NRF2_CSN: track 130.3 -> 127.7 mm, vias 2 -> 1
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
Commit message: Rev 1.2: 18650 battery power (TP4056 + MT3608 + main switch)
- JST-PH 18650 connector, protected TP4056 charger at the left edge
- Main power switch (SW8 + AO3401A), MT3608 boost to 5.3 V, SS34 diode-OR with DevKit USB
- Battery voltage divider on IO3
- Board 116x200 mm; ERC 0/0, DRC 0 (schematic parity), 100% routed

Co-Authored-By: Claude Opus 5.5 <noreply@anthropic.com>
Claude-Session: https://claude.ai/code/session_01M7B8FMVeVb1bqPRBZwSV29
Parts:
- added C18: 100nF, Capacitor_SMD:C_0805_2012Metric_Pad1.18x1.45mm_HandSolder, F.Cu at (75.2, 171.0)
- added D5: SS34, Diode_SMD:D_SMA_Handsoldering, F.Cu at (147.0, 180.5)
- added J10: 18650 BAT, Connector_JST:JST_PH_B2B-PH-K_1x02_P2.00mm_Vertical, F.Cu at (79.5, 152.0)
- added Q4: AO3401A, Package_TO_SOT_SMD:SOT-23, F.Cu at (59.5, 171.0)
- added R19: 100k, Resistor_SMD:R_0805_2012Metric_Pad1.20x1.40mm_HandSolder, F.Cu at (63.2, 171.0)
- added R20: 100k, Resistor_SMD:R_0805_2012Metric_Pad1.20x1.40mm_HandSolder, F.Cu at (68.0, 171.0)
- added R21: 100k, Resistor_SMD:R_0805_2012Metric_Pad1.20x1.40mm_HandSolder, F.Cu at (71.6, 171.0)
- added SW8: MAIN PWR, Button_Switch_THT:SW_Slide_SPDT_Angled_CK_OS102011MA1Q, F.Cu at (49.5, 170.0)
- added U4: TP4056 module (protected), Carrier:TP4056_Module_Pads, F.Cu at (47.5, 148.0)
- added U5: MT3608 boost module (set 5.3V), Carrier:MT3608_Module_Pads, F.Cu at (123.0, 159.0)
- moved BZ1 22.0 mm to (74.5, 218.0)
- moved C16 22.0 mm to (63.5, 213.5)
- moved C17 22.0 mm to (129.4, 202.8)
- moved D4 22.0 mm to (71.5, 227.0)
- moved H3 22.0 mm to (52.0, 225.0)
- moved H4 22.0 mm to (158.0, 225.0)
- moved J9 22.0 mm to (144.6, 209.6)
- moved Q2 22.0 mm to (88.9, 212.5)
- moved Q3 22.0 mm to (58.5, 209.0)
- moved R10 22.0 mm to (62.2, 209.0)
- moved R16 22.0 mm to (58.5, 213.5)
- moved R6 22.0 mm to (89.3, 218.6)
- moved R7 22.0 mm to (89.3, 223.4)
- moved SW1 22.0 mm to (65.2, 178.8)
- moved SW2 22.0 mm to (65.2, 200.8)
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Connections:
- U1 pad 13: unconnected-(U1-IO3-Pad13) -> /BAT_SENSE
Routing:
- net GND: track 624.5 -> 771.5 mm, vias 279 -> 309
- net +5V: track 42.1 -> 151.9 mm, vias 1 -> 2
- net /VBAT_SW: track 0.00 -> 89.7 mm, vias 0 -> 2
- net /BAT_SENSE: track 0.00 -> 54.8 mm, vias 0 -> 1
- net /NRF1_IRQ: track 139.3 -> 187.1 mm, vias 0 -> 2
- net /NRF2_CE: track 123.8 -> 164.4 mm, vias 2 -> 4
- net /VBAT: track 0.00 -> 37.8 mm, vias 0 -> 1
- net /NRF2_IRQ: track 134.5 -> 170.2 mm
- net /CC_CS: track 133.6 -> 167.2 mm
- net /CC_GDO0: track 133.2 -> 165.8 mm
- net +3V3_MOD: track 358.3 -> 389.9 mm, vias 4 -> 2
- net /RFID_TX: track 21.9 -> 51.9 mm, vias 1 -> 0
- net /NRF1_CE: track 91.7 -> 121.0 mm, vias 1 -> 0
- net /IR_RX: track 130.3 -> 158.8 mm, vias 0 -> 1
- net /NRF1_CSN: track 114.3 -> 142.7 mm, vias 0 -> 2
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Other:
- board size 116 x 170 mm -> 116 x 200 mm
- board text added: "BAT ON"
- board text added: "Board 116 x 200 mm"
- board text added: "ESP32-S3 CARRIER v1.2"
- board text removed: "Board 116 x 170 mm"
- board text removed: "ESP32-S3 CARRIER v1.1"
